File: Franklin ACE 1000 Keyboard.kicad_pcb (KiCad board)
At the start: 2 copper layers, 409.8 x 140.5 mm, 84 parts, among them J1 Conn_02x20_Odd_Even, K1 ESC, K10 A, K11 Z, K12 2, K13 W, K14 S, K15 X, K16 3, K17 E, K18 D, K19 C, K2 BREAK, K20 4, K21 R, K22 F, K23 V, K24 5, K25 T, K26 G, K27 B, K28 6, K29 Y, K3 PAUSE, K30 H, K31 N, K32 SPACE, K33 7, K34 U, K35 J, K36 M, K37 8, K38 I, K39 K, K4 CTRL, K40 , / <, K41 9, K42 O, K43 L, K44 . / >, K45 RIGHT, K46 -, K47 +, K48 *, K49 0, K5 TAB, K50 P, K51 ; / :, K52 / ?, K53 7, K54 4, K55 1, K56 >, K57 - / _, K58 [ {, K59 ; ", K6 LOCK, K60 SHIFT, K61 8, K62 5, K63 2, K64 0, K65 + / =, K66 ] }, K67 RETURN, K68 LEFT, K69 9, K7 SHIFT, K70 6, K71 3, K72 ., K8 1, K9 Q

Commit message: Oops, commit actual production board.
Parts:
- K1, K10, K11, K13, K14, K15, K17, K18, K19, K2, K21, K22, K23, K25, K26, K27, K29, K3, K30, K31, K34, K35, K36, K38, K39, K4, K42, K43, K45, K46, K47, K48, K50, K52, K53, K54, K55, K56, K57, K58, K59, K6, K61, K62, K63, K64, K65, K66, K69, K70, K71, K72, K9: footprint Button_Switch_Keyboard:SW_Cherry_MX_1.00u_PCB -> Button_Switch_Keyboard:SW_Cherry_MX_1.00u_Plate
- K12: value 2 -> 2 @; footprint Button_Switch_Keyboard:SW_Cherry_MX_1.00u_PCB -> Button_Switch_Keyboard:SW_Cherry_MX_1.00u_Plate
- K16: value 3 -> 3 #; footprint Button_Switch_Keyboard:SW_Cherry_MX_1.00u_PCB -> Button_Switch_Keyboard:SW_Cherry_MX_1.00u_Plate
- K20: value 4 -> 4 $; footprint Button_Switch_Keyboard:SW_Cherry_MX_1.00u_PCB -> Button_Switch_Keyboard:SW_Cherry_MX_1.00u_Plate
- K24: value 5 -> 5 &; footprint Button_Switch_Keyboard:SW_Cherry_MX_1.00u_PCB -> Button_Switch_Keyboard:SW_Cherry_MX_1.00u_Plate
- K28: value 6 -> 6 ^; footprint Button_Switch_Keyboard:SW_Cherry_MX_1.00u_PCB -> Button_Switch_Keyboard:SW_Cherry_MX_1.00u_Plate
- K32: footprint Button_Switch_Keyboard:SW_Cherry_MX_1.00u_PCB -> Button_Switch_Keyboard:SW_Cherry_MX_6.25u_PCB
- K33: value 7 -> 7 &; footprint Button_Switch_Keyboard:SW_Cherry_MX_1.00u_PCB -> Button_Switch_Keyboard:SW_Cherry_MX_1.00u_Plate
- K37: value 8 -> 8 *; footprint Button_Switch_Keyboard:SW_Cherry_MX_1.00u_PCB -> Button_Switch_Keyboard:SW_Cherry_MX_1.00u_Plate
- K40: value , / < -> , <; footprint Button_Switch_Keyboard:SW_Cherry_MX_1.00u_PCB -> Button_Switch_Keyboard:SW_Cherry_MX_1.00u_Plate
- K41: value 9 -> 9 (; footprint Button_Switch_Keyboard:SW_Cherry_MX_1.00u_PCB -> Button_Switch_Keyboard:SW_Cherry_MX_1.00u_Plate
- K44: value . / > -> . >; footprint Button_Switch_Keyboard:SW_Cherry_MX_1.00u_PCB -> Button_Switch_Keyboard:SW_Cherry_MX_1.00u_Plate
- K49: value 0 -> 0 ); footprint Button_Switch_Keyboard:SW_Cherry_MX_1.00u_PCB -> Button_Switch_Keyboard:SW_Cherry_MX_1.00u_Plate
- K5, K67: footprint Button_Switch_Keyboard:SW_Cherry_MX_1.00u_PCB -> Button_Switch_Keyboard:SW_Cherry_MX_1.50u_Plate
- K51: value ; / : -> ; :; footprint Button_Switch_Keyboard:SW_Cherry_MX_1.00u_PCB -> Button_Switch_Keyboard:SW_Cherry_MX_1.00u_Plate
- K60: footprint Button_Switch_Keyboard:SW_Cherry_MX_1.00u_PCB -> Button_Switch_Keyboard:SW_Cherry_MX_2.00u_Plate
- K68: footprint Button_Switch_Keyboard:SW_Cherry_MX_1.00u_PCB -> Button_Switch_Keyboard:SW_Cherry_MX_1.25u_Plate
- K7: footprint Button_Switch_Keyboard:SW_Cherry_MX_1.00u_PCB -> Button_Switch_Keyboard:SW_Cherry_MX_2.25u_Plate
- K8: value 1 -> 1 !; footprint Button_Switch_Keyboard:SW_Cherry_MX_1.00u_PCB -> Button_Switch_Keyboard:SW_Cherry_MX_1.00u_Plate
- R1: value R_US -> R = (Vcc – Vd) / Id
- moved K6 135.7 mm to (147.4, 197.1)
- moved K52 135.6 mm to (361.7, 216.2)
- moved K62 135.6 mm to (457.0, 178.1)
- moved K11 135.6 mm to (190.3, 216.2)
- moved K13 135.6 mm to (195.1, 178.1)
- moved K17 135.6 mm to (214.2, 178.1)
- moved K23 135.6 mm to (247.4, 216.2)
- moved K25 135.6 mm to (252.3, 178.1)
- moved K27 135.6 mm to (266.5, 216.2)
- moved K28 135.6 mm to (261.8, 159.0)
- moved K29 135.6 mm to (271.4, 178.1)
- moved K30 135.6 mm to (275.4, 197.1)
- moved K33 135.6 mm to (280.8, 159.0)
- moved K35 135.6 mm to (294.4, 197.1)
- moved K61 135.6 mm to (457.0, 159.0)
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Routing:
- net Col6: track 436.1 -> 434.0 mm
- net Net-(D7-K): track 138.8 -> 137.7 mm
- net Net-(D6-K): track 96.5 -> 96.0 mm
- net Col4: track 409.9 -> 409.4 mm
Other:
- board size 409.8 x 140.5 mm -> 410 x 128.5 mm
- board text added: "Franklin ACE 1000 Keyboard (for use with Unified Retro Keyboard ASCII Interface) v0.9 2023 竜 クリストファー (Chris Ryu)"
